File: chess_clock_proj/chess_clock_proj.kicad_sch (KiCad schematic)
At the start: 13 parts

Commit message: conexões feitas
Parts:
- added C? (x2): 22u, symbol Device:C
- added C? (x2): 10p, symbol Device:C
- added D? (x2): GREEN, symbol Device:LED
- added D?: LED, symbol Device:LED
- added D?: RED, symbol Device:LED
- added J? (x2): Conn_01x04_Male, symbol Connector:Conn_01x04_Male
- added R? (x3): 220, symbol Device:R
- added SW? (x2): SW_DIP_x01, symbol Switch:SW_DIP_x01
- added U?: AMS1117-3.3, Package_TO_SOT_SMD:SOT-223-3_TabPin2, symbol Regulator_Linear:AMS1117-3.3
- added Y?: 16MHz, symbol Device:Crystal_GND24
Connections:
- net +3V3: now also C?.1, J?.1 (Pin_1), J?.1 (Pin_1), R?.2, R?.2, R?.2, U?.2 (VO)
- net GND: now also C?.2, C?.2, C?.2, C?.2, J?.4 (Pin_4), J?.4 (Pin_4), SW?.2, SW?.2, U?.1 (GND), Y?.2, Y?.4
- net BUTTON_J1: now reaches U?.10 (PA0)
- net BUTTON_J1: now also SW?.1
- net BUTTON_J2: now reaches U?.11 (PA1)
- net BUTTON_J2: now also SW?.1
- net LED: now reaches U?.2 (PC13)
- net LED: now also D?.1 (K)
- net LED_J1: now reaches U?.21 (PB10)
- net LED_J1: now also D?.1 (K)
- net LED_J2: now reaches U?.22 (PB11)
- net LED_J2: now also D?.1 (K)
- net HSL_IN: now reaches U?.3 (PC14)
- net USART1_TX: now reaches U?.30 (PA9)
- net USART1_TX: now also J?.2 (Pin_2)
- net USART1_RX: now reaches U?.31 (PA10)
- net USART1_RX: now also J?.3 (Pin_3)
- net SWDIO: now reaches U?.34 (PA13)
- net SWDIO: now also J?.2 (Pin_2)
- net SWCLK: now reaches U?.37 (PA14)
- net SWCLK: now also J?.3 (Pin_3)
- net HSL_OUT: now reaches U?.4 (PC15)
- net HSE_IN: now reaches U?.5 (PD0)
- net HSE_IN: now also C?.1, Y?.1
- net HSE_OUT: now reaches U?.6 (PD1)
- net HSE_OUT: now also C?.1, Y?.3
- new net: D?.2 (A), R?.1 (x3)
- new net: C?.1, U?.3 (VI)
- no-connect marks 0 -> 23
Other:
- note added: "1x 100nF per VDD pin (according to the STM32 recommendations)"
- note added: "C = 2*(Cload-Cs) C = 2*(10p-5p) = 10pF"
- note added: "CHESS CLOCK PROJECT - using STM32F103C8T6"
- note added: "LEDS AND SWITCHES OF THE GAME"
- note added: "POWER SUPLY"
- note added: "VDDA Filtering"
